File: mppt-board.kicad_sch (KiCad schematic)
At the start: 28 parts, among them J1 Out, J2 programming, Q1 IPD25N06S4L30ATMA2, U1 MC33201DR2G, U2 LM3671, U3 STM32G030J6Mx

Commit message: init
Parts:
- removed C3: 4.7u, Capacitor_SMD:C_0805_2012Metric, symbol Device:C
- removed C6: 33p, Capacitor_SMD:C_0805_2012Metric, symbol Device:C
- removed C7: 10u, Capacitor_SMD:C_0805_2012Metric, symbol Device:C
- removed J1: Out, Connector_PinSocket_2.54mm:PinSocket_1x02_P2.54mm_Vertical, symbol Connector:Conn_01x02_Socket
- removed L2: 2.2u, Inductor_SMD:L_Vishay_IHLP-1212, symbol Device:L
- removed R6: 562k, Resistor_SMD:R_0805_2012Metric, symbol Device:R
- removed R7: 100k, Resistor_SMD:R_0805_2012Metric, symbol Device:R
- removed SC1: Solar_Cells, Connector_PinHeader_2.54mm:PinHeader_1x02_P2.54mm_Vertical, symbol Device:Solar_Cells
- removed U1: MC33201DR2G, Package_SO:SOIC-8_3.9x4.9mm_P1.27mm, symbol plib:MC33201DR2G
- removed U2: LM3671, Package_TO_SOT_SMD:TSOT-23-5, symbol Regulator_Switching:LM3670MF
- added C4: 0.1u, Capacitor_SMD:C_0805_2012Metric, symbol Device:C
- added U1: INA180A1, Package_TO_SOT_SMD:SOT-23-5, symbol Amplifier_Current:INA180A1
- added U2: LM2937xMP, Package_TO_SOT_SMD:SOT-223-3_TabPin2, symbol Regulator_Linear:LM2937xMP
- added U4: XT60, plib:CONN-TH_XT60, symbol plib:XT60
- added U5: XT60-F, plib:CONN-TH_XT60PB-F, symbol plib:XT60-F
- C5: value 6.8p -> 10u
- D1: footprint Package_TO_SOT_SMD:TO-252-2 -> Package_TO_SOT_SMD:TO-263-2
- L1: value FXL2213-680-M 100u -> MHCI06030-2R2M-R8; footprint plib:IND-SMD_L23.5-W22.0 -> Inductor_SMD:L_Bourns_SRP7028A_7.3x6.6mm
- renumbered C4 to C3
Connections:
- net GND: now also C5.2, C4.2, U1.2 (GND), U2.2 (GND), U5.1
- net VBUS: now also C4.1, U1.5 (V+), U2.1 (VI), U4.2 (+)
- net VCC: now also U2.3 (VO)
- net V_{drop}: now also U1.1
- net at C2.1, D1.2 (K): now also U5.2
- net at R2.2, R4.1: now also U1.3 (+)
- net at R3.2, R5.1: now also U1.4 (-)
- net at R1.1, R2.1: now also U4.1 (-)
